File: PCB/Tinylab_proto1.kicad_pcb (KiCad board)
At the start: 2 copper layers, 36.8 x 34.7 mm, 79 parts, among them IC1 ATXMEGA32A4U-AU, P1 SCOPE_OUT, P10 EXPANSION, P11 SWITCH, P2 USB_OTG, P3 DIG_OUT, P4 PDI/3V3, P5 SCOPE_OUT, P6 DAC_OUT, P7 PSU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

Commit message: Remove PCB label update from PR
Connections:
- IC1 pad 34: /PDI_DATA -> /PDI_CLK
- IC1 pad 35: /PDI_CLK -> /PDI_DATA
- P4 pad 2: /PDI_DATA -> /PDI_CLK
- P4 pad 4: /PDI_CLK -> /PDI_DATA
Routing:
- net /PDI_DATA: track 30.1 -> 27.2 mm
- net /PDI_CLK: track 27.2 -> 30.1 mm
Other:
- net class Default added: clearance 0.2, trace_width 0.25, via_dia 0.6, via_drill 0.4

Commit message: PCB update to swap incorrect labels
Labels for nets PDI_CLK and PDI_DATA swapped to match ATxmega32A4U pinout. saved as Kicad 9.0 files
Connections:
- IC1 pad 34: /PDI_CLK -> /PDI_DATA
- IC1 pad 35: /PDI_DATA -> /PDI_CLK
- P4 pad 2: /PDI_CLK -> /PDI_DATA
- P4 pad 4: /PDI_DATA -> /PDI_CLK
Routing:
- net /PDI_DATA: track 27.2 -> 30.1 mm
- net /PDI_CLK: track 30.1 -> 27.2 mm
Other:
- net class Default removed
